File: monitor-speed/pcb/Comparador_II.kicad_sch (KiCad schematic)
At the start: 25 parts, among them K3 DIPxx-1Cxx-51x, Q4 BC848, U6 TL082, U7 TL082

Commit message: Monitor-Speed: New Schematic
Parts:
- removed C7, C8: 1uF, Capacitor_SMD:C_0603_1608Metric_Pad1.08x0.95mm_HandSolder, symbol Device:C
- removed R23, R24: 100K, Resistor_SMD:R_0603_1608Metric_Pad0.98x0.95mm_HandSolder, symbol Device:R
- removed U6, U7 (x2): TL082, Package_SO:SOIC-8-1EP_3.9x4.9mm_P1.27mm_EP2.29x3mm, symbol Amplifier_Operational:TL082
Connections:
- net +12: no longer R27.1, R32.1
- new net: R27.1, R32.1
Other:
- moved on the sheet: C9, D5, D6, D7, K3, Q4, R25, R26, R27, R28, R29, R30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
