File: monitor-speed/pcb/output_relay.kicad_sch (KiCad schematic)
At the start: 5 parts, among them K2 2961105, Q2 BC848

Commit message: Agregue capas interiores....
Parts:
- renumbered D3 to D10, D4 to D11, K2 to K3, Q2 to Q5, R18 to R35
Changed lines of the file:
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@@
   (symbol (lib_id "power1:+24") (at 138.43 67.945 0)
     (in_bom yes) (on_board yes) (fields_autoplaced)
-    (property "Reference" "#PWR036" (id 0) (at 138.43 66.675 0)
+    (property "Reference" "#PWR038" (id 0) (at 138.43 66.675 0)
       (effects (font (size 0.762 0.762)) hide)
     )
@@
   (symbol (lib_id "power:GND") (at 138.43 117.475 0)
     (in_bom yes) (on_board yes)
-    (property "Reference" "#PWR0122" (id 0) (at 138.43 123.825 0)
+    (property "Reference" "#PWR039" (id 0) (at 138.43 123.825 0)
       (effects (font (size 1.27 1.27)) hide)
     )
@@
   (symbol (lib_id "Device:LED") (at 138.43 108.585 90)
     (in_bom yes) (on_board yes)
-    (property "Reference" "D4" (id 0) (at 141.4272 107.5944 90)
+    (property "Reference" "D11" (id 0) (at 141.4272 107.5944 90)
       (effects (font (size 1.27 1.27)) (justify right))
     )
@@
   (symbol (lib_id "Transistor_BJT:BC848") (at 135.89 97.155 0)
     (in_bom yes) (on_board yes)
-    (property "Reference" "Q2" (id 0) (at 140.7414 95.9866 0)
+    (property "Reference" "Q5" (id 0) (at 140.7414 95.9866 0)
       (effects (font (size 1.27 1.27)) (justify left))
     )
@@
   (symbol (lib_id "Diode:1N4148") (at 138.43 81.915 270)
     (in_bom yes) (on_board yes)
-    (property "Reference" "D3" (id 0) (at 140.462 80.7466 90)
+    (property "Reference" "D10" (id 0) (at 140.462 80.7466 90)
       (effects (font (size 1.27 1.27)) (justify left))
     )
@@
   (symbol (lib_id "eec:2961105") (at 157.48 71.12 270)
     (in_bom yes) (on_board yes) (fields_autoplaced)
-    (property "Reference" "K2" (id 0) (at 161.163 80.3715 90)
+    (property "Reference" "K3" (id 0) (at 161.163 80.3715 90)
       (effects (font (size 1.27 1.27)) (justify left))
     )
@@
   (symbol (lib_id "Device:R") (at 121.92 97.155 90)
     (in_bom yes) (on_board yes)
-    (property "Reference" "R18" (id 0) (at 121.92 91.8972 90))
+    (property "Reference" "R35" (id 0) (at 121.92 91.8972 90))
     (property "Value" "6.8K" (id 1) (at 121.92 94.2086 90))
     (property "Footprint" "Resistor_SMD:R_0603_1608Metric_Pad0.98x0.95mm_HandSolder" (id 2) (at 121.92 98.933 90)
